Commit message: Update utils and add gravity visualization

File: src/robot.urdf (robot description, URDF)
Before this commit: robot linkage, 4 links, 3 joints
Joints:
- joint joint A: origin xyz=0 0 -0.05 -> xyz=0 0 0

Commit message: Add collision detection

File: src/robot.urdf (robot description, URDF)
Before this commit: robot linkage, 4 links, 3 joints
Links:
- removed link link A
- removed link link B
- removed link link C
- added link link_lower_arm, mass 0.5; visual cylinder length=1 radius=0.05
- added link link_sphere, mass 0.5; visual sphere radius=0.05
- added link link_upper_arm, mass 0.5; visual cylinder length=1 radius=0.05
Joints:
- joint joint A: child link B -> link_upper_arm; parent link A -> link_sphere
- joint joint B: child link C -> link_lower_arm; parent link B -> link_upper_arm
- joint joint base: child link A -> link_sphere
