Commit message: Added all pdf's

File: src/robot_heavy.urdf (robot description, URDF)
Before this commit: robot linkage, 4 links, 3 joints
Links:
- link link_lower_arm: mass 10 -> 0.5

Commit message: commit to allow for pulling from github

File: src/robot_heavy.urdf (robot description, URDF)
Before this commit: robot linkage, 4 links, 3 joints
Links:
- link link_lower_arm: mass 0.5 -> 10
